File: PCB/LightShaker-3/LightShaker-3.brd (EAGLE design)
At the start: 221.3 x 25 mm, 75 parts, among them IC1 STM32F042F6P6, IC10 APA102, IC11 APA102, IC12 APA102, IC13 APA102, IC14 APA102, IC15 APA102, IC16 APA102, IC17 APA102, IC18 MAX1765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

Commit message: updated FW for work with Lightshaker-3 HW by adding drvPower to all projects, didn't fix all existing Bugs
Parts:
- added U$2: (no value), DTP_Misc:DOCFIELD
- R19: value 100k -> 10k
- R5: value 56k -> 100k
