File: PCB/LightShaker-3/LightShaker-3.sch (EAGLE design)
At the start: 75 parts, among them IC1 STM32F042F6P6, IC10 APA102, IC11 APA102, IC12 APA102, IC13 APA102, IC14 APA102, IC15 APA102, IC16 APA102, IC17 APA102, IC18 MAX1765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

Commit message: updated FW for work with Lightshaker-3 HW by adding drvPower to all projects, didn't fix all existing Bugs
Parts:
- IC1: PARTNR (none) -> P1480012
- IC18: PARTNR (none) -> P1480011
- IC20: PARTNR (none) -> P1480013
- R10: PARTNR _ -> (none)
- R19: value 100k -> 10k
- R20, R6: PARTNR E0821300_ -> (none)
- R5: value 56k -> 100k; PARTNR E0002800_ -> (none)
Connections:
- net +2V5: now also T3A.S, T3B.S; no longer T3G$1.S, T3G$2.S
- net GATE: now also T3A.G, T3B.G; no longer T3G$1.G, T3G$2.G
- net N$15: now also T3A.D, T3B.D; no longer T3G$1.D, T3G$2.D
Other:
- note removed: "B1962200"
- moved on the sheet: C1, C18, C19, C2, C20, C21, C22, C23, C25, C3, C4, C5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
